File: KiCad/DSP-ADAU1446-core-pcb/PSU.sch (KiCad schematic (older format))
At the start: 0 parts

Commit message: - finished schematics v0.1 - PCB work began - BOM generated
Parts:
- added C30, C32: 0.1uF, w_smd_cap:c_0603, symbol C
- added C31: 10uF, w_smd_cap:c_elec_4x5.3, symbol CP
- added C33, C34: 1uF, w_smd_cap:c_0805, symbol C
- added D1: MBR0530T1G, w_smd_diode:sod123, symbol D_Schottky
- added J1: POW_CONN, w_conn_mkds:mkds_1,5-2, symbol Screw_Terminal_1x02
- added L3: 600R@100MHz, w_smd_inductors:inductor_smd_0603, symbol INDUCTOR
- added R27: 100K, w_smd_resistors:r_0603, symbol R
- added SW1: SW_Push_Dual, w_switch:smd_push2, symbol SW_Push_Dual
- added U3: ADM811RARTZ, w_smd_trans:sot143B, symbol ADM811RARTZ
- added U4, U5: TLV1117LV33, TO_SOT_Packages_SMD:SOT-223-3Lead_TabPin2, symbol NCP1117ST33T3G
Connections:
- new net: D1.2 (A), J1.2
- new net: D1.1 (K), L3.1
- new net GND: C30.1, C31.2, C32.2, C33.2, C34.2, J1.1, R27.2, SW1.1, SW1.3, U3.1 (GND), U4.1 (GND), U5.1 (GND)
- new net VAA: C34.1, U5.2 (VO)
- new net VCC: C31.1, C32.1, L3.2, U4.3 (VI), U5.3 (VI)
- new net VDD: C30.2, C33.1, U3.4 (VCC), U4.2 (VO)
- new net ~BRD_RST: SW1.2, SW1.4, U3.3 (~MR)
- new net ~RESET: R27.1, U3.2 (~RESET)

Commit message: finished schematic and PCB for v0.1
Parts:
- removed SW1: SW_Push_Dual, w_switch:smd_push2, symbol SW_Push_Dual
- added SW1: ALPS_switch, w_switch:smd_push_ALPS, symbol ALPS_switch
Connections:
- net GND: now also SW1.1, SW1.2
- net ~BRD_RST: now also SW1.3, SW1.4
Changed lines of the file:
@@
 ~RESET
-$Comp
-L SW_Push_Dual SW1
-U 1 1 58A189FF
-P 4550 1700
-F 0 "SW1" H 4600 1800 50  0000 L CNN
-F 1 "SW_Push_Dual" H 4550 1430 50  0000 C CNN
-F 2 "w_switch:smd_push2" H 4550 1900 50  0001 C CNN
-F 3 "" H 4550 1900 50  0000 C CNN
-	1    4550 1700
-	1    0    0    -1
-$EndComp
 $Comp
 L GND #PWR042
@@
 Connection ~ 6900 1400
 Wire Wire Line
-	4750 1700 5500 1700
-Wire Wire Line
-	4850 1700 4850 1900
-Wire Wire Line
-	4850 1900 4750 1900
-Connection ~ 4850 1700
+	4750 1900 5200 1900
 Wire Wire Line
 	4000 1700 4350 1700
-Wire Wire Line
-	4250 1700 4250 1900
 Wire Wire Line
 	4250 1900 4350 1900
@@
 Wire Wire Line
 	5200 2150 5200 1700
-Connection ~ 5200 1700
 Wire Wire Line
 	5500 1400 4700 1400
@@
 Wire Wire Line
 	5900 3100 6050 3100
+$Comp
+L ALPS_switch SW1
+U 1 1 58BB62E8
+P 4550 1700
+F 0 "SW1" H 4600 1800 50  0000 L CNN
+F 1 "ALPS_switch" H 4550 1425 50  0000 C CNN
+F 2 "w_switch:smd_push_ALPS" H 4550 1900 50  0000 C CNN
+F 3 "" H 4550 1900 50  0000 C CNN
+	1    4550 1700
+	1    0    0    -1
+$EndComp
+Wire Wire Line
+	5200 1700 5500 1700
+Wire Wire Line
+	4250 1900 4250 1950
+Wire Wire Line
+	4250 1950 4850 1950
+Wire Wire Line
+	4850 1950 4850 1900
+Connection ~ 5200 1900
+Connection ~ 4850 1900
+Wire Wire Line
+	4250 1700 4250 1650
+Wire Wire Line
+	4250 1650 4850 1650
+Wire Wire Line
+	4850 1650 4850 1700
+Wire Wire Line
+	4850 1700 4750 1700
 $EndSCHEMATC
