File: KiCad/DSP-ADAU1446-core-pcb/CONN.sch (KiCad schematic (older format))
At the start: 0 parts

Commit message: - finished schematics v0.1 - PCB work began - BOM generated
Parts:
- added C28, C29: 0.1uF, w_smd_cap:c_0603, symbol C
- added P1: RCA, w_conn_av:rca_yellow, symbol BNC
- added P2, P3, P4, P6, P7: CONN_02x05, w_pin_strip:pin_strip_2mm_5x2, symbol CONN_02X05
- added P5: CONN_02X05, w_pin_strip:pin_strip_2mm_5x2, symbol CONN_02X05
- added R11, R17, R18, R19, R20, R21, R22, R23, R24, R25, R26: 75R, w_smd_resistors:r_0603, symbol R
- added R12, R13, R14, R15: 4K7, w_smd_resistors:r_0603, symbol R
- added R16: 10K, w_smd_resistors:r_0603, symbol R
- added U2: NB3L553, w_smd_dil:msoic-8, symbol NB3L553
Connections:
- new net: P6.4 (P4), R17.1
- new net: P6.6 (P6), R18.1
- new net: P6.8 (P8), R19.1
- new net: P7.4 (P4), R20.1
- new net: P7.6 (P6), R21.1
- new net: P7.8 (P8), R22.1
- new net: P4.2 (P2), R12.2
- new net: P4.4 (P4), R13.2
- new net: P4.6 (P6), R14.2
- new net: P4.8 (P8), R15.2
- new net: R23.2, U2.2 (Q0)
- new net: R24.2, U2.3 (Q1)
- new net: R25.2, U2.6 (Q2)
- new net: R26.2, U2.7 (Q3)
- new net: R16.1, U2.8 (OE)
- new net: C28.2, P1.1 (In), R11.1
- new net BCLK0: P2.6 (P6)
- new net BCLK1: P3.6 (P6)
- new net BCLK2: R18.2
- new net BCLK3: R21.2
- new net CLKOUT: U2.5 (ICLK)
- new net GND: C29.1, P1.2 (Ext), P2.1 (P1), P2.10 (P10), P2.3 (P3), P2.5 (P5), P2.7 (P7), P2.9 (P9), P3.1 (P1), P3.10 (P10), P3.3 (P3), P3.5 (P5), P3.7 (P7), P3.9 (P9), P4.1 (P1), P4.3 (P3), P4.5 (P5), P4.7 (P7), P5.10 (P10), P6.1 (P1), P6.10 (P10), P6.3 (P3), P6.5 (P5), P6.7 (P7), P6.9 (P9), P7.1 (P1), P7.10 (P10), P7.3 (P3), P7.5 (P5), P7.7 (P7), P7.9 (P9), R11.2, U2.4 (GND)
- new net LRCLK0: P2.4 (P4)
- new net LRCLK1: P3.4 (P4)
- new net LRCLK2: R17.2
- new net LRCLK3: R20.2
- new net MCLKA0: P2.2 (P2), R23.1
- new net MCLKA1: P3.2 (P2), R24.1
- new net MCLKD0: P6.2 (P2), R25.1
- new net MCLKD1: P7.2 (P2), R26.1
- new net MP0/ADC0: R12.1
- new net MP1/ADC1: R13.1
- new net MP2/ADC2: R14.1
- new net MP3/ADC3: R15.1
- new net MP4: P4.9 (P9)
- new net MP5: P4.10 (P10)
- new net SCL/CCLK: P5.1 (P1)
- new net SDA/COUT: P5.3 (P3)
- new net SDATA_IN0: P2.8 (P8)
- new net SDATA_IN1: P3.8 (P8)
- new net SDATA_OUT0: R19.2
- new net SDATA_OUT1: R22.2
- new net SPDIFI: C28.1
- new net VDD: C29.2, R16.2, U2.1 (VDD)
- new net ~BRD_RST: P5.6 (P6)
- no-connect marks 0 -> 6
Other:
- note added: "IN CONN"
- note added: "OUT CONN"
- note added: "SPDIF INPUT"

Commit message: -pcb update - changed footprint of IC1 and U2 to SO8
Parts:
- U2: footprint w_smd_dil:msoic-8 -> w_smd_dil:so-8
Changed lines of the file:
@@
 F 0 "U2" H 8950 5850 60  0000 C CNN
 F 1 "NB3L553" H 9100 5750 60  0000 C CNN
-F 2 "w_smd_dil:msoic-8" H 9200 5250 60  0001 C CNN
+F 2 "w_smd_dil:so-8" H 9200 5250 60  0001 C CNN
 F 3 "" H 9200 5250 60  0000 C CNN
 F 4 "NB3L553DG" H 9200 5250 60  0001 C CNN "Mfr. Part No."

Commit message: finished schematic and PCB for v0.1
Parts:
- removed P1: RCA, w_conn_av:rca_yellow, symbol BNC
- added P1: CONN_01X02, Socket_Strips:Socket_Strip_Straight_1x02_Pitch2.54mm, symbol CONN_01X02
Connections:
- net GND: now also P1.2 (P2)
- net LRCLK0: now also P2.8 (P8); no longer P2.4 (P4)
- net LRCLK1: now also P3.8 (P8); no longer P3.4 (P4)
- net SDATA_IN0: now also P2.4 (P4); no longer P2.8 (P8)
- net SDATA_IN1: now also P3.4 (P4); no longer P3.8 (P8)
- net at P4.2 (P2): now also R15.2; no longer R12.2
- net at P4.4 (P4): now also R14.2; no longer R13.2
- net at P4.6 (P6): now also R13.2; no longer R14.2
- net at P4.8 (P8): now also R12.2; no longer R15.2
- net at C28.2, R11.1: now also P1.1 (P1)
Other:
- moved on the sheet: R12, R13, R14, R15
Changed lines of the file:
@@
 	-1   0    0    1
 $EndComp
-Text GLabel 2550 1600 2    60   Input ~ 0
+Text GLabel 2550 2000 2    60   Input ~ 0
 LRCLK0
 Text GLabel 2550 1800 2    60   Input ~ 0
 BCLK0
-Text GLabel 2550 2000 2    60   Input ~ 0
+Text GLabel 2550 1600 2    60   Input ~ 0
 SDATA_IN0
-Text GLabel 2550 3000 2    60   Input ~ 0
+Text GLabel 2550 3400 2    60   Input ~ 0
 LRCLK1
 Text GLabel 2550 3200 2    60   Input ~ 0
 BCLK1
-Text GLabel 2550 3400 2    60   Input ~ 0
+Text GLabel 2550 3000 2    60   Input ~ 0
 SDATA_IN1
 Text GLabel 8900 1600 0    60   Input ~ 0
@@
 L R R13
 U 1 1 589F9B93
+P 6350 1850
+F 0 "R13" V 6430 1850 50  0000 C CNN
+F 1 "4K7" V 6350 1850 50  0000 C CNN
+F 2 "w_smd_resistors:r_0603" V 6280 1850 50  0001 C CNN
+F 3 "" H 6350 1850 50  0000 C CNN
+	1    6350 1850
+	0    1    -1   0
+$EndComp
+$Comp
+L R R14
+U 1 1 589F9BF8
 P 6350 1650
-F 0 "R13" V 6430 1650 50  0000 C CNN
+F 0 "R14" V 6430 1650 50  0000 C CNN
 F 1 "4K7" V 6350 1650 50  0000 C CNN
 F 2 "w_smd_resistors:r_0603" V 6280 1650 50  0001 C CNN
 F 3 "" H 6350 1650 50  0000 C CNN
 	1    6350 1650
-	0    1    1    0
-$EndComp
-$Comp
-L R R14
-U 1 1 589F9BF8
-P 6350 1850
-F 0 "R14" V 6430 1850 50  0000 C CNN
-F 1 "4K7" V 6350 1850 50  0000 C CNN
-F 2 "w_smd_resistors:r_0603" V 6280 1850 50  0001 C CNN
-F 3 "" H 6350 1850 50  0000 C CNN
-	1    6350 1850
-	0    1    1    0
+	0    1    -1   0
 $EndComp
 $Comp
 L R R12
 U 1 1 589F9C35
+P 6350 2050
+F 0 "R12" V 6430 2050 50  0000 C CNN
+F 1 "4K7" V 6350 2050 50  0000 C CNN
+F 2 "w_smd_resistors:r_0603" V 6280 2050 50  0001 C CNN
+F 3 "" H 6350 2050 50  0000 C CNN
+	1    6350 2050
+	0    1    -1   0
+$EndComp
+$Comp
+L R R15
+U 1 1 589F9CA8
 P 6350 1450
-F 0 "R12" V 6430 1450 50  0000 C CNN
+F 0 "R15" V 6430 1450 50  0000 C CNN
 F 1 "4K7" V 6350 1450 50  0000 C CNN
 F 2 "w_smd_resistors:r_0603" V 6280 1450 50  0001 C CNN
 F 3 "" H 6350 1450 50  0000 C CNN
 	1    6350 1450
-	0    1    1    0
-$EndComp
-$Comp
-L R R15
-U 1 1 589F9CA8
-P 6350 2050
-F 0 "R15" V 6430 2050 50  0000 C CNN
-F 1 "4K7" V 6350 2050 50  0000 C CNN
-F 2 "w_smd_resistors:r_0603" V 6280 2050 50  0001 C CNN
-F 3 "" H 6350 2050 50  0000 C CNN
-	1    6350 2050
-	0    1    1    0
-$EndComp
+	0    1    -1   0
+$EndComp
+Text GLabel 6700 2050 2    60   Input ~ 0
+MP0/ADC0
+Text GLabel 6700 1850 2    60   Input ~ 0
+MP1/ADC1
+Text GLabel 6700 1650 2    60   Input ~ 0
+MP2/ADC2
 Text GLabel 6700 1450 2    60   Input ~ 0
-MP0/ADC0
-Text GLabel 6700 1650 2    60   Input ~ 0
-MP1/ADC1
-Text GLabel 6700 1850 2    60   Input ~ 0
-MP2/ADC2
-Text GLabel 6700 2050 2    60   Input ~ 0
 MP3/ADC3
 $Comp
@@
 	2200 1700 2200 1600
 Wire Wire Line
-	2200 1600 2550 1600
-Wire Wire Line
 	1900 1900 2200 1900
 Wire Wire Line
 	2200 1900 2200 2000
 Wire Wire Line
-	2200 2000 2550 2000
-Wire Wire Line
 	2550 3200 1900 3200
 Wire Wire Line
-	2550 3000 2200 3000
-Wire Wire Line
 	2200 3000 2200 3100
 Wire Wire Line
 	2200 3100 1900 3100
 Wire Wire Line
-	2550 3400 2200 3400
-Wire Wire Line
 	2200 3400 2200 3300
 Wire Wire Line
@@
 	5950 2000 5850 2000
 Wire Wire Line
-	6200 2050 6050 2050
-Wire Wire Line
 	6050 2050 6050 1900
 Wire Wire Line
 	6050 1900 5850 1900
 Wire Wire Line
-	6200 1850 6150 1850
-Wire Wire Line
 	6150 1850 6150 1800
 Wire Wire Line
 	6150 1800 5850 1800
 Wire Wire Line
-	6200 1650 6150 1650
-Wire Wire Line
 	6150 1650 6150 1700
 Wire Wire Line
 	6150 1700 5850 1700
 Wire Wire Line
-	6200 1450 6050 1450
-Wire Wire Line
 	6050 1450 6050 1600
 Wire Wire Line
 	6050 1600 5850 1600
 Wire Wire Line
+	6700 1450 6500 1450
+Wire Wire Line
+	6700 1650 6500 1650
+Wire Wire Line
+	6700 1850 6500 1850
+Wire Wire Line
 	6700 2050 6500 2050
-Wire Wire Line
-	6700 1850 6500 1850
-Wire Wire Line
-	6700 1650 6500 1650
-Wire Wire Line
-	6700 1450 6500 1450
 Wire Wire Line
 	6700 2250 5950 2250
@@
 $EndComp
 $Comp
-L BNC P1
-U 1 1 58A241B8
-P 1450 5450
-F 0 "P1" H 1460 5570 50  0000 C CNN
-F 1 "RCA" V 1560 5390 50  0000 C CNN
-F 2 "w_conn_av:rca_yellow" H 1450 5450 50  0001 C CNN
-F 3 "" H 1450 5450 50  0000 C CNN
-	1    1450 5450
-	-1   0    0    -1
-$EndComp
-$Comp
 L R R11
 U 1 1 58A24747
@@
 Connection ~ 8050 4950
 Wire Wire Line
-	1600 5450 3350 5450
-Wire Wire Line
-	1450 5650 1450 5700
+	1350 5450 3350 5450
+Wire Wire Line
+	1450 5550 1450 5700
+Wire Wire Line
+	2200 1600 2550 1600
+Wire Wire Line
+	2200 2000 2550 2000
+Wire Wire Line
+	2200 3000 2550 3000
+Wire Wire Line
+	2200 3400 2550 3400
+$Comp
+L CONN_01X02 P1
+U 1 1 58B17F86
+P 1150 5500
+F 0 "P1" H 1150 5650 50  0000 C CNN
+F 1 "CONN_01X02" V 1250 5500 50  0000 C CNN
+F 2 "Socket_Strips:Socket_Strip_Straight_1x02_Pitch2.54mm" H 1150 5500 50  0001 C CNN
+F 3 "" H 1150 5500 50  0000 C CNN
+	1    1150 5500
+	-1   0    0    -1
+$EndComp
+Wire Wire Line
+	1350 5550 1450 5550
+Wire Wire Line
+	6200 1450 6050 1450
+Wire Wire Line
+	6150 1650 6200 1650
+Wire Wire Line
+	6150 1850 6200 1850
+Wire Wire Line
+	6050 2050 6200 2050
 $EndSCHEMATC

Commit message: Updated schematic and PCB to use SDATA_OUT4 and SDATA_OUT8 with LRCLK4,LRCLK8 and BCLK8,BCLK8
Connections:
- net MCLKD0: now also P7.2 (P2); no longer P6.2 (P2)
- net MCLKD1: now also P6.2 (P2); no longer P7.2 (P2)
- net BCLK2 renamed BCLK4
- net BCLK3 renamed BCLK8
- net LRCLK2 renamed SDATA_OUT4
- net LRCLK3 renamed SDATA_OUT8
- net SDATA_OUT0 renamed LRCLK4
- net SDATA_OUT1 renamed LRCLK8
Changed lines of the file:
@@
 $EndComp
 Text Label 8500 1400 0    60   ~ 0
+MCLKD1
+Text Label 8500 2800 0    60   ~ 0
 MCLKD0
-Text Label 8500 2800 0    60   ~ 0
-MCLKD1
 $Comp
 L GND #PWR034
@@
 Text GLabel 2550 3000 2    60   Input ~ 0
 SDATA_IN1
+Text GLabel 8900 2000 0    60   Input ~ 0
+LRCLK4
+Text GLabel 8900 1800 0    60   Input ~ 0
+BCLK4
 Text GLabel 8900 1600 0    60   Input ~ 0
-LRCLK2
-Text GLabel 8900 1800 0    60   Input ~ 0
-BCLK2
-Text GLabel 8900 2000 0    60   Input ~ 0
-SDATA_OUT0
+SDATA_OUT4
+Text GLabel 8900 3350 0    60   Input ~ 0
+LRCLK8
+Text GLabel 8900 3150 0    60   Input ~ 0
+BCLK8
 Text GLabel 8900 2950 0    60   Input ~ 0
-LRCLK3
-Text GLabel 8900 3150 0    60   Input ~ 0
-BCLK3
-Text GLabel 8900 3350 0    60   Input ~ 0
-SDATA_OUT1
+SDATA_OUT8
 Text GLabel 5000 2000 0    60   Input ~ 0
 MP4
@@
 	2100 2850 2100 3000
 Wire Wire Line
-	8900 1600 9050 1600
-Wire Wire Line
 	8900 1800 9050 1800
 Wire Wire Line
-	8900 2000 9050 2000
-Wire Wire Line
-	8900 2950 9050 2950
-Wire Wire Line
 	8900 3150 9050 3150
-Wire Wire Line
-	8900 3350 9050 3350
 Wire Wire Line
 	5350 2000 5000 2000
@@
 Wire Wire Line
 	6050 2050 6200 2050
+Wire Wire Line
+	9050 2950 8900 2950
+Wire Wire Line
+	9050 3350 8900 3350
+Wire Wire Line
+	8900 1600 9050 1600
+Wire Wire Line
+	8900 2000 9050 2000
 $EndSCHEMATC
